File: Audio_Video.kicad_sch (KiCad schematic)
At the start: 25 parts, among them J6 AudioJack4_SwitchTR1, U1 V3S-split, U10 FPC_40, U9 SY7200AABC

Commit message: PCB done
Parts:
- removed TP8: TestPoint, TestPoint:TestPoint_Pad_D1.0mm, symbol Connector:TestPoint
- added R54, R55: 1R, Resistor_SMD:R_0402_1005Metric, symbol Device:R
- C100: renamed from C85; footprint (none) -> Capacitor_SMD:C_0402_1005Metric; LCSC (none) -> C1525
- C93: renamed from C86; footprint (none) -> LED_SMD:LED_1206_3216Metric; LCSC (none) -> C13585
- C96: renamed from C6; LCSC (none) -> C1525
- C99: renamed from C84; footprint (none) -> Capacitor_SMD:C_0603_1608Metric; LCSC (none) -> C19702
- D17: renamed from D15; footprint (none) -> ESD:ESD5451X-2; LCSC (none) -> C239558
- D18: renamed from D13; footprint (none) -> ESD:ESD5451X-2; LCSC (none) -> C239558
- D19: renamed from D14; footprint (none) -> ESD:ESD5451X-2; LCSC (none) -> C239558
- D23: renamed from D17; footprint Diode_SMD:D_SOD-323 -> Diode_SMD:D_SOD-123; LCSC C191023 -> C8598
- J9: renamed from J6; footprint Connector_Audio:Jack_3.5mm_PJ31060-I_Horizontal -> Connector_Audio:Jack_3.5mm_PJ311_Horizontal; LCSC (none) -> C388632
- L7: renamed from L6; value L -> 4.7uH 1.1A 0.1R; footprint (none) -> Inductor_SMD:L_Bourns-SRN4018; LCSC (none) -> C354574
- R47: renamed from R25; LCSC (none) -> C25105
- R50: renamed from R24; LCSC (none) -> C25105
- R52: renamed from R26; footprint Resistor_SMD:R_0402_1005Metric -> Resistor_SMD:R_0603_1608Metric; LCSC (none) -> C21189
- R53: renamed from R39; footprint (none) -> Resistor_SMD:R_0402_1005Metric; LCSC (none) -> C25744
- R56: renamed from R38; value 1R5 -> 1R; footprint (none) -> Resistor_SMD:R_0402_1005Metric; LCSC (none) -> C25086
- R58: renamed from R27; footprint Resistor_SMD:R_0402_1005Metric -> Resistor_SMD:R_0603_1608Metric; LCSC (none) -> C23345
- R61: renamed from R37; footprint (none) -> Resistor_SMD:R_0402_1005Metric; LCSC (none) -> C25900
- U8: renamed from U1; LCSC (none) -> C2687449
- renumbered TP11 to TP14, TP10 to TP15, TP9 to TP17, TP7 to TP18, U9 to U12
Connections:
- net GND: now also R54.2, R55.2; no longer R56.2
- net at D19.1 (A1), R50.1: now also J9.3; no longer J9.R1
- net at C96.2, D17.1 (A1), R52.1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: now also J9.2; no longer J9.R2
- net at D18.1 (A1), R47.1: now also J9.4; no longer J9.T
- new net: R54.1, R55.1, R56.2
Other:
- moved on the sheet: J9, TP17
