File: Clocks_Buttons.kicad_sch (KiCad schematic)
At the start: 23 parts, among them SW1 SW_Push, SW2 SW_Push, SW3 SW_Push, SW4 SW_Push, U1 V3S-split, Y1 32.768khz, Y2 24MHz

Commit message: PCB done
Parts:
- added C54: 10uF, Capacitor_SMD:C_0603_1608Metric, symbol Device:C
- added C55: 100n, Capacitor_SMD:C_0402_1005Metric, symbol Device:C
- added C60: 10uF/50V, LED_SMD:LED_1206_3216Metric, symbol Device:C
- added D24, D25, D26, D27, D28, D29, D30, D31: LED, LED_SMD:LED_0603_1608Metric, symbol Device:LED
- added D9: 1N5819WS, Diode_SMD:D_SOD-123, symbol Diode:1N5819WS
- added L5: 4.7uH 1.1A 0.1R, Inductor_SMD:L_Bourns-SRN4018, symbol Device:L
- added R27: 4k7, Resistor_SMD:R_0402_1005Metric, symbol Device:R
- added R29: 10R, Resistor_SMD:R_0603_1608Metric, symbol Device:R
- added TP3, TP5, TP7: TestPoint, TestPoint:TestPoint_Pad_D1.0mm, symbol Connector:TestPoint
- added U6: SY7200AABC, Package_TO_SOT_SMD:SOT-23-6, symbol LED_DRIVER:SY7200AABC
- C62: renamed from C3; LCSC (none) -> C1549
- C67: renamed from C8; LCSC (none) -> C1549
- C71: renamed from C4; LCSC (none) -> C1549
- C72: renamed from C7; LCSC (none) -> C1549
- D22: renamed from D3; footprint (none) -> ESD:ESD5451X-2; LCSC (none) -> C239558
- H1, H2, H3, H4: footprint (none) -> MountingHole:MountingHole_3.2mm_M3_ISO7380_Pad
- R42: renamed from R5; LCSC (none) -> C26082
- R48: renamed from R1; footprint (none) -> Resistor_SMD:R_0402_1005Metric; LCSC (none) -> C25741
- R59: renamed from R2; footprint (none) -> Resistor_SMD:R_0402_1005Metric; LCSC (none) -> C25917
- R62: renamed from R15; footprint (none) -> Resistor_SMD:R_0603_1608Metric; LCSC (none) -> C25950
- R63: renamed from R4; footprint (none) -> Resistor_SMD:R_0402_1005Metric; LCSC (none) -> C25744
- R64: renamed from R3; footprint (none) -> Resistor_SMD:R_0402_1005Metric; LCSC (none) -> C25924
- SW5: renamed from SW4; value SW_Push -> A; footprint (none) -> Button_Switch_SMD:SW_SPST_TL3342; LCSC (none) -> C318884
- SW6: renamed from SW3; value SW_Push -> B; footprint (none) -> Button_Switch_SMD:SW_SPST_TL3342; LCSC (none) -> C318884
- SW7: renamed from SW2; value SW_Push -> C; footprint (none) -> Button_Switch_SMD:SW_SPST_TL3342; LCSC (none) -> C318884
- SW8: renamed from SW1; value SW_Push -> D; footprint (none) -> Button_Switch_SMD:SW_SPST_TL3342; LCSC (none) -> C318884
- U8: renamed from U1; LCSC (none) -> C2687449
- Y4: renamed from Y1; LCSC (none) -> C32346; LCSCC C32346 -> (none)
- renumbered TP1 to TP11, Y2 to Y3
Connections:
- net GND: now also C54.2, C55.2, C60.2, R27.2, R29.2, U6.2 (GND)
- new net: D26.1 (K), R29.1, TP7.1, U6.3 (FB)
- new net: D26.2 (A), D28.1 (K)
- new net: D28.2 (A), D30.1 (K)
- new net: D9.2 (A), L5.2, U6.1 (LX)
- new net: C60.1, D24.2 (A), D9.1 (K), TP5.1, U6.5 (OVR)
- new net: D30.2 (A), D31.1 (K)
- new net: D29.1 (K), D31.2 (A)
- new net: D27.1 (K), D29.2 (A)
- new net: D25.1 (K), D27.2 (A)
- new net: D24.1 (K), D25.2 (A)
- new net PWM1: R27.1, TP3.1, U6.4 (EN/PWM)
- new net VCC: C54.1, C55.1, L5.1, U6.6 (VDD)
Other:
- note added: "Backleds"
- note added: "Buttons"
- note added: "Max amps : 20mA R = 200mV / 20mA = 10 Ohms"
- note added: "Mounting holes"
- note added: "V3s Clocks"
- moved on the sheet: D22, H1, H2, H3, H4, R48, R59, R62, R63, R64, SW5, SW6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
