File: Connections.kicad_sch (KiCad schematic)
At the start: 31 parts, among them J1 UART_Header, J2 SERIAL, J3 USB_HOST, J4 RJ45_LED_Shielded, U1 V3S-split, U2 AMS1117-3.3, U3 CH340N, U6 SRV05-4

Commit message: PCB done
Parts:
- added C101, C109, C110: 100n, Capacitor_SMD:C_0402_1005Metric, symbol Device:C
- added C102: 2.2uF, Capacitor_SMD:C_0603_1608Metric, symbol Device:C
- added C103, C107: 1uF, Capacitor_SMD:C_0402_1005Metric, symbol Device:C
- added C104, C105, C106, C108: 4.7uF, Capacitor_SMD:C_0402_1005Metric, symbol Device:C
- added D32: 4148, Diode_SMD:D_SOD-323, symbol Diode:1N4148WS
- added R25, R26: 1k, Resistor_SMD:R_0402_1005Metric, symbol Device:R
- added R65: 4k7, Resistor_SMD:R_0402_1005Metric, symbol Device:R
- added R66: 560k, Resistor_SMD:R_0603_1608Metric, symbol Device:R
- added U13: AMS1117-3.3, Package_TO_SOT_SMD:SOT-223-3_TabPin2, symbol Regulator_Linear:AMS1117-3.3
- added U14: SSD1306_conn, ssd1306:ssd1306_14, symbol SSD1306:SSD1306_conn
- C56: renamed from C1; LCSC (none) -> C1525
- C59: renamed from C2; value 0.1uF -> 100n; LCSC (none) -> C1525
- C61: renamed from C10; LCSC (none) -> C1525
- C70: renamed from C9; LCSC (none) -> C1525
- D10: renamed from D5; value LED -> TX; LCSC (none) -> C2286
- D11: renamed from D4; value LED -> RX; LCSC (none) -> C2286
- D4: renamed from D1; value LED -> SPD; LCSC (none) -> C72038
- D5: renamed from D2; value LED -> LNK; LCSC (none) -> C72043
- FB2: renamed from FB1; LCSC (none) -> C1017
- L6: renamed from L1; footprint Inductor_SMD:L_6.3x6.3_H3 -> Inductor_SMD:L_1206_3216Metric; LCSC (none) -> C1051
- R30: renamed from R19; value 470 -> 1k; footprint Resistor_SMD:R_01005_0402Metric -> Resistor_SMD:R_0402_1005Metric; LCSC (none) -> C11702
- R31: renamed from R20; value 470 -> 1k; footprint Resistor_SMD:R_01005_0402Metric -> Resistor_SMD:R_0402_1005Metric; LCSC (none) -> C11702
- R32: renamed from R8; LCSC (none) -> C23185
- R33: renamed from R7; LCSC (none) -> C23185
- R34: renamed from R14; value 1k -> 220R; LCSC (none) -> C22962
- R35: renamed from R9; LCSC (none) -> C23185
- R36: renamed from R13; LCSC (none) -> C21190
- R37: renamed from R11; value 1K -> 1k; LCSC (none) -> C21190
- R4: renamed from R21; LCSC (none) -> C25792
- R43: renamed from R6; value 6k -> 6k8; footprint Resistor_SMD:R_0603_1608Metric -> Resistor_SMD:R_0402_1005Metric; LCSC (none) -> C25917
- R45: renamed from R12; LCSC (none) -> C21190
- R46: renamed from R10; LCSC (none) -> C23185
- U8: renamed from U1; LCSC (none) -> C2687449
- renumbered J1 to J10, J2 to J5, J4 to J7, J3 to J8, TP2 to TP6, U6 to U11, U3 to U4, U2 to U7
Connections:
- net +3.3V: now also U8.109 (VCC-USB)
- net GND: now also C101.2, C102.1, C104.2, C105.2, C106.1, C108.2, C109.1, C110.1, R66.1, U13.1 (GND), U14.7 (VSS)
- net VCC: now also C101.1, U13.3 (VI)
- net scl: now also U14.10 (SCL)
- net sda: now also U14.11 (SDA)
- net EPHY-TXP: now reaches J7.1, R33.2, U8.92 (EPHY-TXP)
- net EPHY-TXN: now reaches J7.2, R32.2, U8.91 (EPHY-TXN)
- net EPHY-RXP: now reaches J7.3, R35.1, U8.90 (EPHY-RXP)
- net EPHY-RXN: now reaches J7.6, R46.1, U8.89 (EPHY-RXN)
- net at D11.1 (K), J10.4 (Pin_4), U8.49 (PB9/TWI1_SDA/UART0_RX/PB_EINT9): now also R25.1; no longer U4.6 (TXD)
- net at D10.1 (K), J10.5 (Pin_5), U8.48 (PB8/TWI1_SCK/UART0_TX/PB_EINT8): now also R26.2; no longer U4.7 (RXD)
- net USB-D+: now reaches J8.3 (D+), U11.1 (IO1), U8.111 (USB-DP)
- net USB-D-: now reaches J8.2 (D-), U11.3 (IO2), U8.110 (USB-DM)
- net UD+: now reaches J5.3 (D+), U4.1 (UD+)
- net UD-: now reaches J5.2 (D-), U4.2 (UD-)
- net PWM1: now reaches U8.44 (PB5/PWM1/PB_EINT5)
- new net: C106.2, D32.2 (A), R65.2, U14.9 (RES)
- new net: C102.2, U14.13 (VCOMH)
- new net: R25.2, U4.6 (TXD)
- new net: R66.2, U14.12 (IREF)
- new net: C107.2, U14.1 (C2P)
- new net: C108.1, C109.2, U14.14 (VCC)
- new net: C107.1, U14.2 (C2N)
- new net: C103.2, U14.3 (C1P)
- new net: C103.1, U14.4 (C1N)
- new net: C104.1, C105.1, C110.2, D32.1 (K), R65.1, U13.2 (VO), U14.5 (VBAT), U14.8 (VDD)
- new net: R26.1, U4.7 (RXD)
Other:
- note added: "0.91" OLED"
- moved on the sheet: J10, J8, R33, U11
