File: Memory.kicad_sch (KiCad schematic)
At the start: 30 parts, among them J5 Micro_SD_Card, U1 V3S-split, U4 W25Q128JVS, U5 FEMDRM008G-58A39_NO_NC

Commit message: PCB done
Parts:
- removed J5: Micro_SD_Card, Connector_Card:microSD_HC_Molex_104031-0811, symbol Connector:Micro_SD_Card
- removed RN1: 10k, Resistor_SMD:R_Array_Concave_4x0402, symbol Device:R_Network04
- added C58: 10uF, Capacitor_SMD:C_0603_1608Metric, symbol Device:C
- added J6: 47352-1001, 47352-1001:MOLEX_47352-1001, symbol 47352-1001:47352-1001
- added R39, R40, R41, R44: 10k, Resistor_SMD:R_0402_1005Metric, symbol Device:R
- C57: renamed from C12; footprint Capacitor_SMD:C_0603_1608Metric -> Capacitor_SMD:C_0402_1005Metric; LCSC (none) -> C1525
- C85: renamed from C15; value 0.1uF -> 100n; LCSC (none) -> C1525
- C92: renamed from C14; value 0.1uF -> 100n; LCSC (none) -> C1525
- C94: renamed from C17; value 3.3uF -> 4.7uF; LCSC (none) -> C23733
- C95: renamed from C5; LCSC (none) -> C1525
- C97: renamed from C16; value 3.3uF -> 4.7uF; LCSC (none) -> C23733
- C98: renamed from C13; value C -> 1uF; LCSC (none) -> C52923
- D12: renamed from D11; footprint (none) -> ESD:ESD5451X-2; LCSC (none) -> C239558
- D13: renamed from D8; footprint (none) -> ESD:ESD5451X-2; LCSC (none) -> C239558
- D14: renamed from D10; footprint (none) -> ESD:ESD5451X-2; LCSC (none) -> C239558
- D15: renamed from D9; footprint (none) -> ESD:ESD5451X-2; LCSC (none) -> C239558
- D16: renamed from D6; footprint (none) -> ESD:ESD5451X-2; LCSC (none) -> C239558
- D20: renamed from D12; footprint (none) -> ESD:ESD5451X-2; LCSC (none) -> C239558
- D21: renamed from D7; footprint (none) -> ESD:ESD5451X-2; LCSC (none) -> C239558
- R24: renamed from R46; LCSC (none) -> C25744
- R28: renamed from R16; LCSC (none) -> C25744
- R49: renamed from R22; LCSC (none) -> C25105
- R51: renamed from R17; LCSC (none) -> C25744
- R57: renamed from R23; LCSC (none) -> C25744
- R60: renamed from R18; LCSC (none) -> C25744
- U5: renamed from U4; value W25Q128JVS -> SPI FLASH
- U8: renamed from U1; LCSC (none) -> C2687449
- U9: renamed from U5; value FEMDRM008G-58A39_NO_NC -> eMMC 8GB
- renumbered RN2 to RN1, TP6 to TP10, TP5 to TP13, TP3 to TP16
Connections:
- net +3.3V: now also C58.1, J6.4 (VDD), R39.1, R40.1, R41.1, R44.1
- net GND: now also C58.2, J6.6 (VSS), J6.S1 (SHIELD), J6.S2 (SHIELD), J6.S3 (SHIELD), J6.S4 (SHIELD)
- net at D21.1 (A1), R57.2, U8.101 (PF5/SDC0_D2/JTAG_CK1): now also J6.1 (DATA2)
- net at D13.1 (A1), U8.102 (PF4/SDC0_D3/UART0_RX): now also J6.2 (CD/DATA3), R41.2
- net at D15.1 (A1), U8.103 (PF3/SDC0_CMD/JTAG_DO1): now also J6.3 (CMD), R44.2
- net at D16.1 (A1), R49.1: now also J6.5 (CLK)
- net at D14.1 (A1), U8.106 (PF1/SDC0_D0/JTAG_DI1): now also J6.7 (DATA0), R39.2
- net at D12.1 (A1), U8.107 (PF0/SDC0_D1/JTAG_MS1): now also J6.8 (DATA1), R40.2
- no-connect marks 6 -> 7
