File: Power.kicad_sch (KiCad schematic)
At the start: 99 parts, among them J7 USB_POWER, J8 Bat, SW6 SW_Push, SW7 SW_SPDT, U1 V3S-split, U11 AXP209, U8 SY8088AAC

Commit message: PCB done
Parts:
- removed C69: 100uF, Capacitor_SMD:C_0402_1005Metric, symbol Device:C
- removed SW7: SW_SPDT, Button_Switch_SMD:SW_DIP_SPSTx01_Slide_6.7x4.1mm_W6.73mm_P2.54mm_LowProfile_JPin, symbol Switch:SW_SPDT
- removed TP13: TestPoint, TestPoint:TestPoint_Pad_D1.0mm, symbol Connector:TestPoint
- removed U8: SY8088AAC, Package_TO_SOT_SMD:SOT-23-5, symbol FunKey:SY8088AAC
- added C6: 100uF, Capacitor_Tantalum_SMD:CP_EIA-3528-21_Kemet-B, symbol Device:C_Polarized
- added C79: 100n, Capacitor_SMD:C_0402_1005Metric, symbol Device:C
- added D2: 3.3, LED_SMD:LED_0603_1608Metric, symbol Device:LED
- added D3: PWR, LED_SMD:LED_0603_1608Metric, symbol Device:LED
- added R6: 1k, Resistor_SMD:R_0603_1608Metric, symbol Device:R
- added R8: 2k2, Resistor_SMD:R_0402_1005Metric, symbol Device:R
- added SW2: POWER, Button_Switch_SMD:SW_SPST_TL3342, symbol Switch:SW_Push
- added U1: SY8088AAC, Package_TO_SOT_SMD:SOT-23-5, symbol Allwinner:SY8088AAC
- C1: renamed from C33; value 10n -> 10nF; LCSC (none) -> C15195
- C10: renamed from C62; LCSC (none) -> C1523
- C11: renamed from C77; LCSC (none) -> C1546
- C12: renamed from C52; LCSC (none) -> C15525
- C13: renamed from C56; LCSC (none) -> C15525
- C14: renamed from C80; LCSC (none) -> C23733
- C16: renamed from C81; LCSC (none) -> C15525
- C17: renamed from C67; value 10u -> 10uF; LCSC (none) -> C15525
- C18: renamed from C68; LCSC (none) -> C52923
- C19: renamed from C78; LCSC (none) -> C52923
- C2: renamed from C63; LCSC (none) -> C15525
- C20: renamed from C61; LCSC (none) -> C15525
- C21: renamed from C55; LCSC (none) -> C1525
- C22: renamed from C57; LCSC (none) -> C52923
- C23: renamed from C75; LCSC (none) -> C15525
- C24: renamed from C70; value 4.7u -> 4.7uF; LCSC (none) -> C23733
- C25: renamed from C76; LCSC (none) -> C15525
- C26: renamed from C66; LCSC (none) -> C15525
- C27: renamed from C82; LCSC (none) -> C19702
- C28: renamed from C73; value 0.22uF -> 220nF; LCSC (none) -> C16772
- C29: renamed from C72; LCSC (none) -> C52923
- C3: renamed from C64; LCSC (none) -> C1523
- C30: renamed from C58; LCSC (none) -> C23733
- C31: renamed from C74; LCSC (none) -> C15525
- C32: renamed from C59; LCSC (none) -> C23733
- C33: renamed from C53; LCSC (none) -> C1525
- C34: renamed from C83; value 0.22uF -> 220nF; LCSC (none) -> C16772
- C35: renamed from C65; LCSC (none) -> C15525
- C37: renamed from C41; LCSC (none) -> C1525
- C39: renamed from C47; LCSC (none) -> C1525
- C4: renamed from C71; LCSC (none) -> C1546
- C40: renamed from C50; LCSC (none) -> C1525
- C41: renamed from C42; LCSC (none) -> C1525
- C43: renamed from C29; LCSC (none) -> C1525
- C44: renamed from C19; value 10u -> 10uF; LCSC (none) -> C15525
- C48: renamed from C43; LCSC (none) -> C1525
- C5: renamed from C45; value 10u -> 10uF; LCSC (none) -> C15525
- C50: renamed from C46; LCSC (none) -> C1525
- C51: renamed from C31; LCSC (none) -> C1525
- C52: renamed from C36; LCSC (none) -> C1525
- C63: renamed from C26; value 1u -> 1uF; LCSC (none) -> C52923
- C64: renamed from C44; LCSC (none) -> C1525
- C65: renamed from C32; LCSC (none) -> C1525
- C66: renamed from C28; value 1u -> 1uF; LCSC (none) -> C52923
- C68: renamed from C39; value 1u -> 1uF; LCSC (none) -> C52923
- C69: renamed from C21; value 10u -> 10uF; LCSC (none) -> C15525
- C7: renamed from C49; LCSC (none) -> C1525
- C73: renamed from C20; value 1u -> 1uF; LCSC (none) -> C52923
- C74: renamed from C37; LCSC (none) -> C1525
- C75: renamed from C51; LCSC (none) -> C1525
- C76: renamed from C48; LCSC (none) -> C1525
- C77: renamed from C35; LCSC (none) -> C1525
- C78: renamed from C38; LCSC (none) -> C1525
- C8: renamed from C60; LCSC (none) -> C23733
- C80: renamed from C11; value 10u -> 10uF; LCSC (none) -> C15525
- C81: renamed from C34; LCSC (none) -> C1525
- C82: renamed from C27; LCSC (none) -> C1525
- C83: renamed from C30; value 1u -> 1uF; LCSC (none) -> C52923
- C84: renamed from C22; LCSC (none) -> C1525
- C86: renamed from C23; value 1u -> 1uF; LCSC (none) -> C52923
- C87: renamed from C40; value 10u -> 10uF; LCSC (none) -> C15525
- C88: renamed from C24; value 1u -> 1uF; LCSC (none) -> C52923
- C89: renamed from C25; value 1u -> 1uF; LCSC (none) -> C52923
- C9: renamed from C79; LCSC (none) -> C15525
- C90: renamed from C54; LCSC (none) -> C23733
- C91: renamed from C18; value 10u -> 10uF; LCSC (none) -> C15525
- D1: renamed from D16; value LED -> CHRG; LCSC (none) -> C2286
- D6: renamed from D18; value D_Schottky -> 1N5819WS; footprint (none) -> Diode_SMD:D_SOD-123
- J3: renamed from J8; value Bat -> BATT
- J4: renamed from J7; value USB_POWER -> POWER
- L1: renamed from L4; footprint Inductor_SMD:L_6.3x6.3_H3 -> Inductor_SMD:L_Bourns-SRN4018; LCSC (none) -> C354574
- L2: renamed from L3; footprint Inductor_SMD:L_6.3x6.3_H3 -> Inductor_SMD:L_Bourns-SRN4018; LCSC (none) -> C354574
- L3: renamed from L5; footprint Inductor_SMD:L_6.3x6.3_H3 -> Inductor_SMD:L_Bourns-SRN4018; LCSC (none) -> C354574
- L4: renamed from L2; footprint Inductor_SMD:L_6.3x6.3_H3 -> Inductor_SMD:L_Bourns-SRN4018; LCSC (none) -> C354574
- R1: renamed from R36; footprint Resistor_SMD:R_01005_0402Metric -> Resistor_SMD:R_0402_1005Metric; LCSC (none) -> C11702
- R10: renamed from R40; footprint Resistor_SMD:R_0402_1005Metric -> Resistor_SMD:R_0603_1608Metric; LCSC (none) -> C21189
- R11: renamed from R33; footprint (none) -> Resistor_SMD:R_0402_1005Metric; LCSC (none) -> C25764
- R12: renamed from R44; footprint Resistor_SMD:R_01005_0402Metric -> Resistor_SMD:R_0402_1005Metric; LCSC (none) -> C25792
- R13: renamed from R41; footprint Resistor_SMD:R_0603_1608Metric -> Resistor_SMD:R_1206_3216Metric; LCSC (none) -> C245439
- R14: renamed from R32; footprint (none) -> Resistor_SMD:R_0402_1005Metric; LCSC (none) -> C25741
- R15: renamed from R31; footprint (none) -> Resistor_SMD:R_0402_1005Metric; LCSC (none) -> C4109
- R16: renamed from R30; footprint (none) -> Resistor_SMD:R_0402_1005Metric; LCSC (none) -> C4109
- R2: renamed from R43; footprint Resistor_SMD:R_01005_0402Metric -> Resistor_SMD:R_0805_2012Metric; LCSC (none) -> C17539
- R3: renamed from R42; footprint Resistor_SMD:R_01005_0402Metric -> Resistor_SMD:R_0402_1005Metric; LCSC (none) -> C11702
- R38: renamed from R35; footprint (none) -> Resistor_SMD:R_0603_1608Metric; LCSC (none) -> C23350
- R5: renamed from R29; LCSC (none) -> C25792
- R7: renamed from R45; value 10k -> 2k2; footprint Resistor_SMD:R_01005_0402Metric -> Resistor_SMD:R_0402_1005Metric; LCSC (none) -> C25879
- R9: renamed from R34; footprint (none) -> Resistor_SMD:R_0402_1005Metric; LCSC (none) -> C25741
- SW1: renamed from SW6; value SW_Push -> RESET; footprint (none) -> Button_Switch_SMD:SW_SPST_TL3342; LCSC (none) -> C318884
- U2: renamed from U11; LCSC (none) -> C2997895
- U8: renamed from U1; LCSC (none) -> C2687449
- renumbered TP17 to TP12, TP14 to TP2, TP16 to TP8, TP15 to TP9
Connections:
- net +3.3V: now also C79.1, R6.2
- net +VDC: now also R8.1
- net GND: now also C6.2, C79.2, D2.1 (K), D3.1 (K), SW2.2, U1.2 (GND)
- net VCC: now also U1.4 (VIN)
- net at U2.30 (BACKUP): now also C6.1
- net at R14.2: now also U1.1 (EN)
- net at L4.1: now also U1.3 (LX)
- net at C33.2, R11.2, R9.1: now also U1.5 (FB)
- net at R3.1: now also SW2.1
- new net: D3.2 (A), R8.2
- new net: D2.2 (A), R6.1
- no-connect marks 7 -> 6
Other:
- note added: "Vcc-usb"
- moved on the sheet: J4, R5
