File: STM32.kicad_sch (KiCad schematic)
At the start: 25 parts, among them J10 Conn_02x12_Odd_Even, J9 Conn_02x05_Odd_Even, SW5 SW_Push, SW8 SW_SPDT, U7 STM32F030C8Tx, Y3 32.768khz, Y4 16MHz

Commit message: PCB done
Parts:
- removed J10: Conn_02x12_Odd_Even, symbol Connector_Generic:Conn_02x12_Odd_Even
- removed J9: Conn_02x05_Odd_Even, symbol Connector_Generic:Conn_02x05_Odd_Even
- removed R49, R50: 2k2, symbol Device:R
- removed SW8: SW_SPDT, Button_Switch_SMD:SW_DIP_SPSTx01_Slide_6.7x4.1mm_W6.73mm_P2.54mm_LowProfile_JPin, symbol Switch:SW_SPDT
- added D7, D8: LED, LED_SMD:LED_0603_1608Metric, symbol Device:LED
- added J1: Conn_02x16_Odd_Even, Connector_PinHeader_2.54mm:PinHeader_2x16_P2.54mm_Vertical_SMD, symbol Connector_Generic:Conn_02x16_Odd_Even
- added J2: SWD, Connector_PinHeader_2.54mm:PinHeader_2x02_P2.54mm_Vertical, symbol Connector_Generic:Conn_01x04
- added R17: 220R, Resistor_SMD:R_0402_1005Metric, symbol Device:R
- added R21: 1k, Resistor_SMD:R_0402_1005Metric, symbol Device:R
- added SW4: BOOT, Button_Switch_SMD:SW_SPST_TL3342, symbol Switch:SW_Push
- C15: renamed from C87; value 12pf -> 12pF; LCSC (none) -> C1547
- C36: renamed from C89; LCSC (none) -> C1549
- C38: renamed from C90; LCSC (none) -> C1549
- C42: renamed from C94; LCSC (none) -> C23733
- C45: renamed from C93; LCSC (none) -> C23733
- C46: renamed from C88; value 12pf -> 12pF; LCSC (none) -> C1547
- C47: renamed from C92; value 100pf -> 100pF; LCSC (none) -> C1546
- C49: renamed from C91; value 100pf -> 100pF; LCSC (none) -> C1546
- C53: renamed from C95; value 100pf -> 100pF; LCSC (none) -> C1546
- FB1: renamed from FB2; LCSC (none) -> C1017
- R18: renamed from R48; footprint (none) -> Resistor_SMD:R_0402_1005Metric; LCSC (none) -> C25744
- R19: renamed from R47; footprint (none) -> Resistor_SMD:R_0402_1005Metric; LCSC (none) -> C25118
- R20: renamed from R28; footprint (none) -> Resistor_SMD:R_0402_1005Metric; LCSC (none) -> C25744
- R22: renamed from R52; footprint (none) -> Resistor_SMD:R_0402_1005Metric; LCSC (none) -> C25879
- R23: renamed from R51; footprint (none) -> Resistor_SMD:R_0402_1005Metric; LCSC (none) -> C25879
- SW3: renamed from SW5; value SW_Push -> RST; footprint (none) -> Button_Switch_SMD:SW_SPST_TL3342; LCSC (none) -> C318884
- U3: renamed from U7; value STM32F030C8Tx -> STM32
- Y2: renamed from Y3; LCSC (none) -> C32346; LCSCC C32346 -> (none)
- renumbered TP12 to TP1, Y4 to Y1
Connections:
- net +3.3V: now also J1.31 (Pin_31), SW4.2
- net GND: now also R18.1, J1.2 (Pin_2), J2.1 (Pin_1), R17.2, R21.2
- net I2C2_SCL: now also J1.14 (Pin_14)
- net I2C2_SDA: now also J1.13 (Pin_13)
- net NRST: now also J2.3 (Pin_3)
- net PWM_CH1: now also D8.2 (A)
- net SWCLK: now also J2.2 (Pin_2)
- net SWDIO: now also J2.4 (Pin_4)
- net USART1_RX: now also J1.19 (Pin_19)
- net USART1_TX: now also J1.20 (Pin_20)
- net USART2_RX: now also J1.6 (Pin_6)
- net USART2_TX: now also J1.3 (Pin_3)
- net PA1: now reaches U3.11 (PA1)
- net PA1: now also J1.4 (Pin_4)
- net PA4: now reaches U3.14 (PA4)
- net PA4: now also J1.5 (Pin_5)
- net PB0: now reaches U3.18 (PB0)
- net PB0: now also J1.9 (Pin_9)
- net PB1: now reaches U3.19 (PB1)
- net PB1: now also J1.12 (Pin_12)
- net PC13: now reaches U3.2 (PC13)
- net PC13: now also J1.1 (Pin_1)
- net PB2: now reaches U3.20 (PB2)
- net PB2: now also J1.11 (Pin_11)
- net PB12: now reaches U3.25 (PB12)
- net PB12: now also J1.16 (Pin_16)
- net PB13: now reaches U3.26 (PB13)
- net PB13: now also J1.15 (Pin_15)
- net PB14: now reaches U3.27 (PB14)
- net PB14: now also J1.18 (Pin_18)
- net PB15: now reaches U3.28 (PB15)
- net PB15: now also J1.17 (Pin_17)
- net PA11: now reaches U3.32 (PA11)
- net PA11: now also J1.22 (Pin_22)
- net PA12: now reaches U3.33 (PA12)
- net PA12: now also J1.21 (Pin_21)
- net PF6: now reaches U3.35 (PF6)
- net PF6: now also J1.24 (Pin_24)
- net PF7: now reaches U3.36 (PF7)
- net PF7: now also J1.23 (Pin_23)
- net PA15: now reaches U3.38 (PA15)
- net PA15: now also J1.30 (Pin_30)
- net PB3: now reaches U3.39 (PB3)
- net PB3: now also J1.29 (Pin_29)
- net PB4: now reaches U3.40 (PB4)
- net PB4: now also J1.28 (Pin_28)
- net PB5: now reaches U3.41 (PB5)
- net PB5: now also J1.27 (Pin_27)
- net at U3.44 (BOOT0): now also R18.2, SW4.1; no longer R18.1
- net PB8: now reaches U3.45 (PB8)
- net PB8: now also J1.26 (Pin_26)
- net PB9: now reaches U3.46 (PB9)
- net PB9: now also J1.25 (Pin_25)
- net ADC0 renamed ACT_LED
- net ACT_LED: now also D7.2 (A)
- net I2C1_SCL renamed scl
- net I2C1_SDA renamed sda
- net SPI1_MISO renamed PA6
- net PA6: now also J1.7 (Pin_7)
- net SPI1_MOSI renamed PA7
- net PA7: now also J1.10 (Pin_10)
- net SPI1_SCK renamed PA5
- net PA5: now also J1.8 (Pin_8)
- new net: D8.1 (K), R17.1
- new net: D7.1 (K), R21.1
- new net VCC: J1.32 (Pin_32)
- no-connect marks 34 -> 0
Other:
- moved on the sheet: R18, R22, R23, TP1
