File: lb_mp1.kicad_sch (KiCad schematic)
At the start: 94 parts, among them J1 USB_POWER, J9 Bat, SW1 SW_Push, SW2 SW_SPDT, U1 V3S-split, U3 SY8088AAC, U8 AXP209

Commit message: cleaning and naming
Parts:
- removed C2, C21, C5, C59, C6, C72, C75: 10u, Capacitor_SMD:C_0402_1005Metric, symbol Device:C
- removed C20, C38, C44, C45, C46, C48, C50, C58: 1u, Capacitor_SMD:C_0402_1005Metric, symbol Device:C
- removed C22, C24, C26, C27, C39, C40, C41, C42, C76, C79, C82: 10uF, Capacitor_SMD:C_0402_1005Metric, symbol Device:C
- removed C23, C25: 1nF, Capacitor_SMD:C_0402_1005Metric, symbol Device:C
- removed C28, C47, C49, C51, C52, C53, C54, C55, C56, C57, C60, C61, C62, C63, C64, C65, C66, C67, C68, C73, C77, C78: 100n, Capacitor_SMD:C_0402_1005Metric, symbol Device:C
- removed C29, C33, C36, C80: 1uF, Capacitor_SMD:C_0402_1005Metric, symbol Device:C
- removed C30, C31, C32, C69, C81: 4.7uF, Capacitor_SMD:C_0402_1005Metric, symbol Device:C
- removed C34: 100uF, Capacitor_SMD:C_0402_1005Metric, symbol Device:C
- removed C35: 4.7u, Capacitor_SMD:C_0402_1005Metric, symbol Device:C
- removed C37, C43: 0.22uF, Capacitor_SMD:C_0402_1005Metric, symbol Device:C
- removed C70, C74: 100pF, Capacitor_SMD:C_0402_1005Metric, symbol Device:C
- removed C71: 10n, Capacitor_SMD:C_0402_1005Metric, symbol Device:C
- removed C83: 10uF, Capacitor_SMD:C_0603_1608Metric, symbol Device:C
- removed D5: LED, LED_SMD:LED_0603_1608Metric, symbol Device:LED
- removed D6: D_Schottky, symbol Device:D_Schottky
- removed J1: USB_POWER, Connector_USB:USB_Micro-B_Molex-105017-0001, symbol Connector:USB_B_Micro
- removed J9: Bat, Connector_Molex:Molex_PicoBlade_53047-0310_1x03_P1.25mm_Vertical, symbol Connector_Generic:Conn_01x02
- removed L2, L3, L4, L5: 4.7uH 1.1A 0.1R, Inductor_SMD:L_6.3x6.3_H3, symbol Device:L
- removed R22: 240R, symbol Device:R
- removed R23, R29: 1k, Resistor_SMD:R_01005_0402Metric, symbol Device:R
- removed R24: 47k, Resistor_SMD:R_01005_0402Metric, symbol Device:R
- removed R25: 47k, Resistor_SMD:R_0402_1005Metric, symbol Device:R
- removed R26: 200k 1%, Resistor_SMD:R_01005_0402Metric, symbol Device:R
- removed R27: 0.03R, Resistor_SMD:R_0603_1608Metric, symbol Device:R
- removed R28: 10k, Resistor_SMD:R_01005_0402Metric, symbol Device:R
- removed R3, R4: 2k, symbol Device:R
- removed R30, R32: 100k, symbol Device:R
- removed R31: 200k, symbol Device:R
- removed R46: 0R, Resistor_SMD:R_0402_1005Metric, symbol Device:R
- removed SW1: SW_Push, symbol Switch:SW_Push
- removed SW2: SW_SPDT, Button_Switch_SMD:SW_DIP_SPSTx01_Slide_6.7x4.1mm_W6.73mm_P2.54mm_LowProfile_JPin, symbol Switch:SW_SPDT
- removed U1: V3S-split, Allwinner:V3s-ELQFP-128, symbol Allwinner:V3S-split
- removed U3: SY8088AAC, Package_TO_SOT_SMD:SOT-23-5, symbol FunKey:SY8088AAC
- removed U8: AXP209, Allwinner:AXP209-QFN48, symbol Allwinner:AXP209
Connections:
- no-connect marks 7 -> 0
Other:
- sheet Untitled Sheet renamed Clocks Buttons
- sheet Untitled Sheet2 renamed Connections
- sheet Untitled Sheet3 renamed Memory
- sheet Untitled Sheet4 renamed Audio Video
- sheet Untitled Sheet5 renamed STM32
- added sheet Power (Power.kicad_sch)
- sheet Audio Video: file untitled4.kicad_sch -> Audio_Video.kicad_sch
- sheet Clocks Buttons: file untitled.kicad_sch -> Clocks_Buttons.kicad_sch
- sheet Connections: file untitled2.kicad_sch -> Connections.kicad_sch
- sheet Memory: file untitled3.kicad_sch -> Memory.kicad_sch
- sheet STM32: file untitled5.kicad_sch -> STM32.kicad_sch
- note removed: "0-1"
- note removed: "0-5"
- note removed: "2-3"
- note removed: "4"
- note removed: "5"
- note removed: "6"
- note removed: "7"
- note removed: "8-11"
- note removed: "Avcc"
- note removed: "Ephy-vcc"
- note removed: "Ephy-vdd"
- note removed: "Vcc-mcsi"
- note removed: "Vcc-pe"
- note removed: "Vcc-pll"
- note removed: "Vcc-rtc"
- note removed: "Vcpu"
- note removed: "Vio"
- note removed: "Vram"
- note removed: "Vsys"
- title: (none) -> OzzyBoard

Commit message: PCB done
Other:
- sheet Clocks Buttons renamed Clocks Buttons - lights
