File: hardware/RevB/Audio_Video.kicad_sch (KiCad schematic)
At the start: 30 parts, among them J9 AudioJack4_SwitchTR1, U10 FPC_40, U12 SY7200AABC, U7 NS2009, U8 V3S-split

Commit message: Removed gerber files, reajusted paths for files, added photo and PDF
Other:
- title: OzzyBoard -> OzzyBoard Rev B
Changed lines of the file:
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@@
   (paper "A4")
   (title_block
-    (title "OzzyBoard")
-    (date "2023-03-10")
-    (rev "0.91")
+    (title "OzzyBoard Rev B")
+    (date "2024-01-15")
+    (rev "0.92")
   )
   (junction (at 113.03 163.83) (diameter 0) (color 0 0 0 0)
