File: hardware/RevB/Clocks_Buttons.kicad_sch (KiCad schematic)
At the start: 63 parts, among them J12 tooling_hole, J13 tooling_hole, J14 tooling_hole, SW5 A, SW6 B, SW7 C, SW8 D, U15 74HC595, U6 SY7200AABC, U8 V3S-split, Y3 24MHz, Y4 32.768khz

Commit message: Removed gerber files, reajusted paths for files, added photo and PDF
Other:
- title: OzzyBoard -> OzzyBoard Rev B
Changed lines of the file:
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@@
   (paper "A4")
   (title_block
-    (title "OzzyBoard")
-    (date "2023-03-10")
-    (rev "0.91")
+    (title "OzzyBoard Rev B")
+    (date "2024-01-15")
+    (rev "0.92")
   )
   (junction (at 215.9 46.99) (diameter 0) (color 0 0 0 0)
