File: hardware/RevB/Connections.kicad_sch (KiCad schematic)
At the start: 40 parts, among them J10 UART_Header, J5 SERIAL, J7 RJ45_LED_Shielded, J8 USB_HOST, U11 SRV05-4, U14 SSD1306_conn, U4 CH340N, U8 V3S-split

Commit message: Removed gerber files, reajusted paths for files, added photo and PDF
Other:
- title: OzzyBoard -> OzzyBoard Rev B
Changed lines of the file:
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@@
   (paper "A4")
   (title_block
-    (title "OzzyBoard")
-    (date "2023-03-10")
-    (rev "0.91")
+    (title "OzzyBoard Rev B")
+    (date "2024-01-15")
+    (rev "0.92")
   )
   (junction (at 71.12 96.52) (diameter 0) (color 0 0 0 0)
