File: hardware/RevB/Memory.kicad_sch (KiCad schematic)
At the start: 36 parts, among them J6 Molex-5033981892, U13 EEPROM, U5 SPI FLASH, U8 V3S-split, U9 eMMC

Commit message: Removed gerber files, reajusted paths for files, added photo and PDF
Other:
- title: OzzyBoard -> OzzyBoard Rev B
Changed lines of the file:
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@@
   (paper "A4")
   (title_block
-    (title "OzzyBoard")
-    (date "2023-03-10")
-    (rev "0.91")
+    (title "OzzyBoard Rev B")
+    (date "2024-01-15")
+    (rev "0.92")
   )
   (junction (at 199.39 60.96) (diameter 0) (color 0 0 0 0)
