File: hardware/RevB/Power.kicad_sch (KiCad schematic)
At the start: 106 parts, among them J11 DC POWER, J3 BATT, J4 POWER, SW1 RESET, SW2 POWER, U1 SY8088AAC, U2 AXP209, U8 V3S-split

Commit message: Removed gerber files, reajusted paths for files, added photo and PDF
Other:
- title: OzzyBoard -> OzzyBoard Rev B
Changed lines of the file:
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@@
   (paper "A3")
   (title_block
-    (title "OzzyBoard")
-    (date "2023-03-10")
-    (rev "0.91")
+    (title "OzzyBoard Rev B")
+    (date "2024-01-15")
+    (rev "0.92")
   )
   (junction (at 153.67 138.43) (diameter 0) (color 0 0 0 0)
