File: hardware/RevB/STM32.kicad_sch (KiCad schematic)
At the start: 28 parts, among them J1 Conn_02x16_Odd_Even, J2 SWD, SW3 RST, SW4 BOOT, SW9 FUNC, U3 STM32, Y1 16MHz, Y2 32.768khz

Commit message: Removed gerber files, reajusted paths for files, added photo and PDF
Other:
- title: OzzyBoard -> OzzyBoard Rev B
Changed lines of the file:
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@@
   (paper "A4")
   (title_block
-    (title "OzzyBoard")
-    (date "2023-03-10")
-    (rev "0.91")
+    (title "OzzyBoard Rev B")
+    (date "2024-01-15")
+    (rev "0.92")
   )
   (junction (at 39.37 26.67) (diameter 0) (color 0 0 0 0)
