File: hardware/RevB/lb_mp1.kicad_sch (KiCad schematic)
At the start: 0 parts

Commit message: Removed gerber files, reajusted paths for files, added photo and PDF
Other:
- title: OzzyBoard -> OzzyBoard Rev B
Changed lines of the file:
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@@
   (paper "A3")
   (title_block
-    (title "OzzyBoard")
-    (date "2023-03-10")
-    (rev "0.91")
+    (title "OzzyBoard Rev B")
+    (date "2024-01-15")
+    (rev "0.92")
   )
   (sheet (at 316.23 154.94) (size 55.88 57.15) (fields_autoplaced)
